File: hw/puntel.sch (KiCad schematic (older format))
At the start: 49 parts, among them J1 UEXT, J2 STRIP-3, J3 USB-power, J4 USB-prog, J5 STRIP-4, J6 STRIP-4, Q1 DTA114, SW1 BUTTON, SW2 BUTTON, U1 AP2111H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

Commit message: hw: routed (without uext)
Signed-off-by: Alessandro Rubini <rubini@gnudd.com>
Parts:
- removed J1: UEXT, ~, symbol UEXT
Connections:
- net labels removed: SDA1
- wire segments 202 -> 190
Changed lines of the file:
@@
 Wire Wire Line
 	6475 3200 6675 3200
-$Comp
-L UEXT J1
-U 1 1 596C8205
-P 1100 2575
-F 0 "J1" H 1100 2275 60  0000 C CNN
-F 1 "UEXT" H 1100 2925 60  0000 C CNN
-F 2 "~" H 1100 2575 60  0000 C CNN
-F 3 "~" H 1100 2575 60  0000 C CNN
-	1    1100 2575
-	1    0    0    -1
-$EndComp
 Text Label 3275 1250 0    40   ~ 0
 RST*
-Wire Wire Line
-	1200 2325 1250 2325
-Wire Wire Line
-	1250 2325 1250 2025
-Wire Wire Line
-	1200 2375 1300 2375
-Wire Wire Line
-	1300 2375 1300 3025
-$Comp
-L GND #PWR012
-U 1 1 596C8210
-P 1300 3025
-F 0 "#PWR012" H 1300 3025 30  0001 C CNN
-F 1 "GND" H 1300 2955 30  0001 C CNN
-F 2 "" H 1300 3025 60  0000 C CNN
-F 3 "" H 1300 3025 60  0000 C CNN
-	1    1300 3025
-	1    0    0    -1
-$EndComp
-Wire Wire Line
-	1200 2425 1500 2425
-Wire Wire Line
-	1200 2475 1650 2475
-Wire Wire Line
-	1200 2525 1800 2525
-Wire Wire Line
-	1200 2575 1950 2575
-Wire Wire Line
-	1500 2625 1200 2625
-Wire Wire Line
-	1200 2675 1700 2675
-Wire Wire Line
-	1200 2725 1850 2725
-Wire Wire Line
-	1200 2775 2000 2775
-Text Label 1350 2425 0    40   ~ 0
-TXD
-Text Label 1550 2475 0    40   ~ 0
-RXD
-Text Label 1700 2525 0    40   ~ 0
-SCL
-Text Label 1850 2575 0    40   ~ 0
-SDA
-Text Label 1350 2625 0    40   ~ 0
-MISO
-Text Label 1550 2675 0    40   ~ 0
-MOSI
-Text Label 1700 2725 0    40   ~ 0
-SCK
-Text Label 1850 2775 0    40   ~ 0
-SSEL
 Text Label 3275 3150 0    40   ~ 0
 TXD
@@
 Connection ~ 5675 725
 $Comp
-L GND #PWR013
+L GND #PWR012
 U 1 1 596C8252
 P 5325 1025
-F 0 "#PWR013" H 5325 1025 30  0001 C CNN
+F 0 "#PWR012" H 5325 1025 30  0001 C CNN
 F 1 "GND" H 5325 955 30  0001 C CNN
 F 2 "" H 5325 1025 60  0000 C CNN
@@
 $EndComp
 $Comp
-L GND #PWR014
+L GND #PWR013
 U 1 1 596C8258
 P 5675 1025
-F 0 "#PWR014" H 5675 1025 30  0001 C CNN
+F 0 "#PWR013" H 5675 1025 30  0001 C CNN
 F 1 "GND" H 5675 955 30  0001 C CNN
 F 2 "" H 5675 1025 60  0000 C CNN
@@
 NoConn ~ 3525 3250
 NoConn ~ 3525 2950
-NoConn ~ 3525 2450
 NoConn ~ 3525 2350
 NoConn ~ 3525 1950
@@
 DM
 $Comp
-L +3.3V #PWR015
+L +3.3V #PWR014
 U 1 1 596C8287
 P 6825 2100
-F 0 "#PWR015" H 6825 2060 30  0001 C CNN
+F 0 "#PWR014" H 6825 2060 30  0001 C CNN
 F 1 "+3.3V" H 6825 2210 30  0000 C CNN
 F 2 "" H 6825 2100 60  0001 C CNN
@@
 	4625 850  4825 850
 $Comp
-L +3.3V #PWR016
+L +3.3V #PWR015
 U 1 1 596C8290
 P 6125 725
-F 0 "#PWR016" H 6125 685 30  0001 C CNN
+F 0 "#PWR015" H 6125 685 30  0001 C CNN
 F 1 "+3.3V" H 6125 835 30  0000 C CNN
 F 2 "" H 6125 725 60  0001 C CNN
@@
 Connection ~ 2875 1700
 $Comp
-L +3.3V #PWR017
+L +3.3V #PWR016
 U 1 1 596C82A6
 P 2700 1450
-F 0 "#PWR017" H 2700 1410 30  0001 C CNN
+F 0 "#PWR016" H 2700 1410 30  0001 C CNN
 F 1 "+3.3V" H 2700 1560 30  0000 C CNN
 F 2 "" H 2700 1450 60  0001 C CNN
@@
 $EndComp
 $Comp
-L +3.3V #PWR018
+L +3.3V #PWR017
 U 1 1 596C82B2
 P 6425 4100
-F 0 "#PWR018" H 6425 4060 30  0001 C CNN
+F 0 "#PWR017" H 6425 4060 30  0001 C CNN
 F 1 "+3.3V" H 6425 4210 30  0000 C CNN
 F 2 "" H 6425 4100 60  0001 C CNN
@@
 	2700 1550 3525 1550
 Connection ~ 2700 1550
-$Comp
-L +3.3V #PWR019
-U 1 1 596C82C2
-P 1250 2025
-F 0 "#PWR019" H 1250 1985 30  0001 C CNN
-F 1 "+3.3V" H 1250 2135 30  0000 C CNN
-F 2 "" H 1250 2025 60  0001 C CNN
-F 3 "" H 1250 2025 60  0001 C CNN
-	1    1250 2025
-	1    0    0    -1
-$EndComp
 Wire Wire Line
 	3525 2550 3250 2550
+Text Label 3300 2650 0    40   ~ 0
+RLED
+Wire Wire Line
+	3525 2450 3250 2450
 Text Label 3300 2550 0    40   ~ 0
-RLED
-Wire Wire Line
-	6200 2550 5925 2550
-Text Label 5975 2550 0    40   ~ 0
 YLED
 NoConn ~ 5925 1250
@@
 Connection ~ 1350 1325
 $Comp
-L GND #PWR020
+L GND #PWR018
 U 1 1 596C8993
 P 1350 1475
-F 0 "#PWR020" H 1350 1475 30  0001 C CNN
+F 0 "#PWR018" H 1350 1475 30  0001 C CNN
 F 1 "GND" H 1350 1405 30  0001 C CNN
 F 2 "" H 1350 1475 60  0000 C CNN
@@
 Wire Wire Line
 	3250 2650 3525 2650
-Text Label 3300 2650 0    40   ~ 0
+Text Label 3300 2450 0    40   ~ 0
 GLED
 $Comp
@@
 	2700 2975 2700 3125
 $Comp
-L GND #PWR021
+L GND #PWR019
 U 1 1 596C8C83
 P 2700 3125
-F 0 "#PWR021" H 2700 3125 30  0001 C CNN
+F 0 "#PWR019" H 2700 3125 30  0001 C CNN
 F 1 "GND" H 2700 3055 30  0001 C CNN
 F 2 "" H 2700 3125 60  0000 C CNN
@@
 	9825 4550 9825 6775
 $Comp
-L +5V #PWR022
+L +5V #PWR020
 U 1 1 596C8FF6
 P 9825 4550
-F 0 "#PWR022" H 9825 4640 20  0001 C CNN
+F 0 "#PWR020" H 9825 4640 20  0001 C CNN
 F 1 "+5V" H 9825 4640 30  0000 C CNN
 F 2 "" H 9825 4550 60  0000 C CNN
@@
 	10750 4875 10750 7025
 $Comp
-L GND #PWR023
+L GND #PWR021
 U 1 1 596C94DB
 P 10750 7025
-F 0 "#PWR023" H 10750 7025 30  0001 C CNN
+F 0 "#PWR021" H 10750 7025 30  0001 C CNN
 F 1 "GND" H 10750 6955 30  0001 C CNN
 F 2 "" H 10750 7025 60  0000 C CNN
@@
 Connection ~ 10325 3550
 $Comp
-L +5V #PWR024
+L +5V #PWR022
 U 1 1 596C9C93
 P 10325 3350
-F 0 "#PWR024" H 10325 3440 20  0001 C CNN
+F 0 "#PWR022" H 10325 3440 20  0001 C CNN
 F 1 "+5V" H 10325 3440 30  0000 C CNN
 F 2 "" H 10325 3350 60  0000 C CNN
@@
 $EndComp
 $Comp
-L GND #PWR025
+L GND #PWR023
 U 1 1 596C9CA2
 P 10325 4050
-F 0 "#PWR025" H 10325 4050 30  0001 C CNN
+F 0 "#PWR023" H 10325 4050 30  0001 C CNN
 F 1 "GND" H 10325 3980 30  0001 C CNN
 F 2 "" H 10325 4050 60  0000 C CNN
@@
 $EndComp
 $Comp
-L +3.3V #PWR026
+L +3.3V #PWR024
 U 1 1 596D0A82
 P 2550 5475
-F 0 "#PWR026" H 2550 5435 30  0001 C CNN
+F 0 "#PWR024" H 2550 5435 30  0001 C CNN
 F 1 "+3.3V" H 2550 5585 30  0000 C CNN
 F 2 "" H 2550 5475 60  0001 C CNN
@@
 	1450 5725 1750 5725
 $Comp
-L GND #PWR027
+L GND #PWR025
 U 1 1 596D0A8E
 P 1650 6175
-F 0 "#PWR027" H 1650 6175 30  0001 C CNN
+F 0 "#PWR025" H 1650 6175 30  0001 C CNN
 F 1 "GND" H 1650 6105 30  0001 C CNN
 F 2 "" H 1650 6175 60  0000 C CNN
@@
 	1650 6025 1650 6175
 $Comp
-L GND #PWR028
+L GND #PWR026
 U 1 1 596D0A96
 P 2600 6175
-F 0 "#PWR028" H 2600 6175 30  0001 C CNN
+F 0 "#PWR026" H 2600 6175 30  0001 C CNN
 F 1 "GND" H 2600 6105 30  0001 C CNN
 F 2 "" H 2600 6175 60  0000 C CNN
@@
 	3550 7000 3550 7300
 $Comp
-L +3.3V #PWR029
+L +3.3V #PWR027
 U 1 1 596D0ABA
 P 3550 6550
-F 0 "#PWR029" H 3550 6510 30  0001 C CNN
+F 0 "#PWR027" H 3550 6510 30  0001 C CNN
 F 1 "+3.3V" H 3550 6660 30  0000 C CNN
 F 2 "" H 3550 6550 60  0001 C CNN
@@
 Connection ~ 4050 7300
 $Comp
-L GND #PWR030
+L GND #PWR028
 U 1 1 596D0AE5
 P 4050 7400
-F 0 "#PWR030" H 4050 7400 30  0001 C CNN
+F 0 "#PWR028" H 4050 7400 30  0001 C CNN
 F 1 "GND" H 4050 7330 30  0001 C CNN
 F 2 "" H 4050 7400 60  0000 C CNN
@@
 $EndComp
 $Comp
-L +3.3V #PWR031
+L +3.3V #PWR029
 U 1 1 596D0AEB
 P 5150 6550
-F 0 "#PWR031" H 5150 6510 30  0001 C CNN
+F 0 "#PWR029" H 5150 6510 30  0001 C CNN
 F 1 "+3.3V" H 5150 6660 30  0000 C CNN
 F 2 "" H 5150 6550 60  0001 C CNN
@@
 EEPROM: Bus address 0x57 (ae/af)
 $Comp
-L +3.3V #PWR032
+L +3.3V #PWR030
 U 1 1 596D0AF8
 P 1375 6975
-F 0 "#PWR032" H 1375 6935 30  0001 C CNN
+F 0 "#PWR030" H 1375 6935 30  0001 C CNN
 F 1 "+3.3V" H 1375 7085 30  0000 C CNN
 F 2 "" H 1375 6975 60  0001 C CNN
@@
 	1375 7225 1375 7275
 $Comp
-L GND #PWR033
+L GND #PWR031
 U 1 1 596D0B08
 P 1375 7275
-F 0 "#PWR033" H 1375 7275 30  0001 C CNN
+F 0 "#PWR031" H 1375 7275 30  0001 C CNN
 F 1 "GND" H 1375 7205 30  0001 C CNN
 F 2 "" H 1375 7275 60  0000 C CNN
@@
 	2875 7025 2875 7175
 $Comp
-L GND #PWR034
+L GND #PWR032
 U 1 1 596D0B10
 P 2875 7175
-F 0 "#PWR034" H 2875 7175 30  0001 C CNN
+F 0 "#PWR032" H 2875 7175 30  0001 C CNN
 F 1 "GND" H 2875 7105 30  0001 C CNN
 F 2 "" H 2875 7175 60  0000 C CNN
@@
 $EndComp
 $Comp
-L +3.3V #PWR035
+L +3.3V #PWR033
 U 1 1 596D0B16
 P 2625 6875
-F 0 "#PWR035" H 2625 6835 30  0001 C CNN
+F 0 "#PWR033" H 2625 6835 30  0001 C CNN
 F 1 "+3.3V" H 2625 6985 30  0000 C CNN
 F 2 "" H 2625 6875 60  0001 C CNN
@@
 NoConn ~ 5000 5400
 Text Label 5200 5700 0    40   ~ 0
-SDA1
+SDA
 $Comp
 L CSMALL C8
@@
 	3600 5300 4200 5300
 $Comp
-L +3.3V #PWR036
+L +3.3V #PWR034
 U 1 1 596D1393
 P 3775 5200
-F 0 "#PWR036" H 3775 5160 30  0001 C CNN
+F 0 "#PWR034" H 3775 5160 30  0001 C CNN
 F 1 "+3.3V" H 3775 5310 30  0000 C CNN
 F 2 "" H 3775 5200 60  0000 C CNN
@@
 Connection ~ 3875 5825
 $Comp
-L GND #PWR037
+L GND #PWR035
 U 1 1 596D13B1
 P 3875 5925
-F 0 "#PWR037" H 3875 5925 30  0001 C CNN
+F 0 "#PWR035" H 3875 5925 30  0001 C CNN
 F 1 "GND" H 3875 5855 30  0001 C CNN
 F 2 "" H 3875 5925 60  0000 C CNN
@@
 	5425 5300 5425 5350
 $Comp
-L GND #PWR038
+L GND #PWR036
 U 1 1 596D13B8
 P 5425 5350
-F 0 "#PWR038" H 5425 5350 30  0001 C CNN
+F 0 "#PWR036" H 5425 5350 30  0001 C CNN
 F 1 "GND" H 5425 5280 30  0001 C CNN
 F 2 "" H 5425 5350 60  0000 C CNN
@@
 	5125 5500 5125 5200
 $Comp
-L +3.3V #PWR039
+L +3.3V #PWR037
 U 1 1 596D13BF
 P 5125 5200
-F 0 "#PWR039" H 5125 5160 30  0001 C CNN
+F 0 "#PWR037" H 5125 5160 30  0001 C CNN
 F 1 "+3.3V" H 5125 5310 30  0000 C CNN
 F 2 "" H 5125 5200 60  0000 C CNN
@@
 	1    0    0    -1
 $EndComp
-Text Label 5250 5600 0    40   ~ 0
+Text Label 5200 5600 0    40   ~ 0
 SCL
 Wire Wire Line
@@
 Magnetometer: Bus address 0x0e (1c/1d)
 $Comp
-L +5V #PWR040
+L +5V #PWR038
 U 1 1 596D02D3
 P 8125 5950
-F 0 "#PWR040" H 8125 6040 20  0001 C CNN
+F 0 "#PWR038" H 8125 6040 20  0001 C CNN
 F 1 "+5V" H 8125 6040 30  0000 C CNN
 F 2 "" H 8125 5950 60  0000 C CNN
@@
 	1    0    0    -1
 $EndComp
+NoConn ~ 5925 2550
 $EndSCHEMATC

Commit message: hw: beautify schematic file (no change)
Signed-off-by: Alessandro Rubini <rubini@gnudd.com>
Parts:
- J4: value USB-prog -> USB-comm
Other:
- note added: "3.3V Regulator"
- note added: "Diagnostic Leds"
- note added: "I2C Peripherals\n"
- note added: "Microcontroller"
- note added: "Pixels"
- note added: "Side Connectors"
- note added: "USB Power and Communication\n"
- note added: "User Buttons"
- note removed: "3.3V"
- note removed: "Misc-out"
- moved on the sheet: C1, C2, D1, D2, D3, D4, J2, J5, J6, JS1, L1, Q1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
